File: hardware/schakelklok/schakelklok.sch (KiCad schematic (older format))
At the start: 9 parts

Commit message: finished schematic
Parts:
- added D? (x4): LED, symbol Device:LED
- added Q? (x5): BD439, Package_TO_SOT_THT:TO-126-3_Vertical, symbol Transistor_BJT:BD439
- added R? (x7): 2k, symbol Device:R_Small
- added R? (x5): 200, symbol Device:R_Small
- added RV?: R_POT_TRIM, symbol Device:R_POT_TRIM
- added U?: 24LC64, symbol Memory_EEPROM:24LC64
- R? (x2): value R -> 2k
- R?: value R -> 10k
Connections:
- net labels added: D4, D5, D6, D7, SCL, SDA, chip_enable, display_light, enable, interrupt_request, miso1, mosi1, nss1, pulse_A, pulse_b, push, readwrite, register_select, schakeluitgang_1, schakeluitgang_2, schakeluitgang_3, schakeluitgang_4, sck1
- wire segments 64 -> 139
- no-connect marks 0 -> 1

Commit message: started routing
Parts:
- added J2: schakeluitgangen, Connector_PinHeader_2.54mm:PinHeader_1x04_P2.54mm_Vertical, symbol Connector_Generic:Conn_01x04
- added J3: programmer_1, Connector_PinHeader_2.54mm:PinHeader_1x04_P2.54mm_Vertical, symbol Connector_Generic:Conn_01x04
- added J4: programmer_2, Connector_PinHeader_2.54mm:PinHeader_1x04_P2.54mm_Vertical, symbol Connector_Generic:Conn_01x04
- D1, D2, D3, D4: renamed from D?; footprint (none) -> LED_THT:LED_D5.0mm
- DS1: footprint harms_usual:16x02LCD_display -> harms_usual:lcd24x2
- J1: renamed from J?; footprint (none) -> Connector_PinHeader_2.54mm:PinHeader_1x04_P2.54mm_Vertical
- R1, R10, R11, R12, R13, R14, R15, R2, R3, R4, R5, R6, R7, R8, R9: renamed from R?; footprint (none) -> harms_usual:Resistor_Horizontal_RM7mm
- RV1: renamed from RV?; footprint (none) -> Potentiometer_THT:Potentiometer_Bourns_3266Y_Vertical
- SW1: renamed from SW?; footprint (none) -> Rotary_Encoder:RotaryEncoder_Alps_EC11E-Switch_Vertical_H20mm
- U1: renamed from U?; footprint (none) -> harms_usual:DIP-8_W7.62mm_LongPads
- U2: renamed from U?; footprint (none) -> harms_usual:DIP-40_W15.24mm_LongPads
- U3: renamed from U?; footprint (none) -> harms_usual:nrf24l01
- gave numbers to parts that had none: 5
Connections:
- net schakeluitgang_1: now also J2.1 (Pin_1)
- net schakeluitgang_2: now also J2.2 (Pin_2)
- net schakeluitgang_3: now also J2.3 (Pin_3)
- net schakeluitgang_4: now also J2.4 (Pin_4)
- new net: J3.1 (Pin_1), J4.1 (Pin_1)
- new net: J3.2 (Pin_2), J4.2 (Pin_2)
- new net: J3.3 (Pin_3), J4.3 (Pin_3)
- new net: J3.4 (Pin_4), J4.4 (Pin_4)

Commit message: finished hardware
Parts:
- removed J2: schakeluitgangen, Connector_PinHeader_2.54mm:PinHeader_1x04_P2.54mm_Vertical, symbol Connector_Generic:Conn_01x04
- added J2: Conn_01x05, Connector_PinHeader_2.54mm:PinHeader_1x05_P2.54mm_Vertical, symbol Connector_Generic:Conn_01x05
Connections:
- net GND: now also J2.5 (Pin_5)
- net schakeluitgang_1: now also J2.1 (Pin_1)
- net schakeluitgang_2: now also J2.2 (Pin_2)
- net schakeluitgang_3: now also J2.3 (Pin_3)
- net schakeluitgang_4: now also J2.4 (Pin_4)
- no-connect marks 1 -> 11
Changed lines of the file:
@@
 encoding utf-8
 Sheet 1 1
-Title ""
-Date ""
-Rev ""
-Comp ""
+Title "embedded control "
+Date "2020-09-12"
+Rev "0"
+Comp "Harm Hongerkamp"
 Comment1 ""
 Comment2 ""
@@
 Wire Wire Line
 	5400 4600 5300 4600
-$Comp
-L Connector_Generic:Conn_01x04 J2
-U 1 1 5F5E2A92
-P 7400 6050
-F 0 "J2" V 7272 6230 50  0000 L CNN
-F 1 "schakeluitgangen" V 7363 6230 50  0000 L CNN
-F 2 "Connector_PinHeader_2.54mm:PinHeader_1x04_P2.54mm_Vertical" H 7400 6050 50  0001 C CNN
-F 3 "~" H 7400 6050 50  0001 C CNN
-	1    7400 6050
-	0    1    1    0
-$EndComp
 Text GLabel 7500 5850 1    50   Input ~ 0
 schakeluitgang_1
@@
 Wire Wire Line
 	5000 5750 5000 5450
+NoConn ~ 3550 2700
+NoConn ~ 3550 2800
+NoConn ~ 3550 2900
+NoConn ~ 3550 3000
+NoConn ~ 5300 3800
+NoConn ~ 5300 3700
+NoConn ~ 5300 3400
+NoConn ~ 4400 4100
+NoConn ~ 4400 4300
+$Comp
+L Connector_Generic:Conn_01x05 J2
+U 1 1 5F6DA5D6
+P 7300 6050
+F 0 "J2" V 7172 6330 50  0000 L CNN
+F 1 "Conn_01x05" V 7263 6330 50  0000 L CNN
+F 2 "Connector_PinHeader_2.54mm:PinHeader_1x05_P2.54mm_Vertical" H 7300 6050 50  0001 C CNN
+F 3 "~" H 7300 6050 50  0001 C CNN
+	1    7300 6050
+	0    1    1    0
+$EndComp
+$Comp
+L power:GND #PWR01
+U 1 1 5F6DBD2F
+P 6950 5850
+F 0 "#PWR01" H 6950 5600 50  0001 C CNN
+F 1 "GND" H 6955 5677 50  0000 C CNN
+F 2 "" H 6950 5850 50  0001 C CNN
+F 3 "" H 6950 5850 50  0001 C CNN
+	1    6950 5850
+	1    0    0    -1
+$EndComp
+Wire Wire Line
+	6950 5850 6950 5800
+Wire Wire Line
+	6950 5800 7100 5800
+Wire Wire Line
+	7100 5800 7100 5850
+NoConn ~ 21850 6850
 $EndSCHEMATC
